File: KiCadFiles/FullAdder/FullAdder.kicad_pcb (KiCad board)
At the start: 2 copper layers, 139.7 x 94 mm, 45 parts, among them Q1 Q_NPN_CBE, Q2 Q_NPN_CBE, Q3 Q_NPN_CBE, Q4 Q_NPN_CBE, Q5 Q_NPN_CBE, Q6 Q_NPN_CBE, Q7 Q_NPN_CBE, Q8 Q_NPN_CBE, Q9 Q_NPN_CBE

Commit message: updated design
Parts:
- added D19: D, Diode_THT:D_DO-35_SOD27_P2.54mm_Vertical_KathodeUp, F.Cu at (109.2, 48.3)
- added D20: D, Diode_THT:D_DO-35_SOD27_P2.54mm_Vertical_KathodeUp, F.Cu at (104.1, 53.3)
- added D21: D, Diode_THT:D_DO-35_SOD27_P2.54mm_Vertical_KathodeUp, F.Cu at (116.8, 48.3)
- added D22: D, Diode_THT:D_DO-35_SOD27_P2.54mm_Vertical_KathodeUp, F.Cu at (121.9, 53.3)
- added R19: 10k, Resistor_THT:R_Axial_DIN0309_L9.0mm_D3.2mm_P2.54mm_Vertical, F.Cu at (109.2, 53.3)
- added R20: 10k, Resistor_THT:R_Axial_DIN0309_L9.0mm_D3.2mm_P2.54mm_Vertical, F.Cu at (114.3, 53.3)
- moved R12 23.4 mm to (124.5, 58.4), turned to 180 degrees
- moved R10 23.0 mm to (101.6, 58.4), turned to 0 degrees
- moved D14 3.59 mm to (121.9, 55.9), turned to 180 degrees
- moved D11 3.59 mm to (109.2, 55.9), turned to 180 degrees
- moved Q6 3.59 mm to (111.8, 58.4), turned to 180 degrees
- moved R8 2.65 mm to (101.6, 50.9)
- moved D10 2.54 mm to (104.1, 40.6)
- moved D13 2.54 mm to (121.9, 40.6)
- moved Q5 2.54 mm to (111.8, 50.8)
- moved Q7 2.54 mm to (114.3, 50.8)
- moved R11 2.54 mm to (124.5, 50.8)
- moved D12 2.54 mm to (109.2, 43.2), turned to 180 degrees
- moved D15 2.54 mm to (116.8, 43.2), turned to 0 degrees
Connections:
- Q5 pad 2: Net-(D10-Pad2) -> Net-(Q5-Pad2)
- Q5 pad 3: Net-(D11-Pad2) -> Net-(Q5-Pad3)
- Q7 pad 2: Net-(D13-Pad2) -> Net-(Q7-Pad2)
- Q7 pad 3: Net-(D14-Pad2) -> Net-(Q7-Pad3)
- R11 pad 2: Net-(D14-Pad2) -> Net-(Q7-Pad3)
- R8 pad 2: Net-(D11-Pad2) -> Net-(Q5-Pad3)
Routing:
- net GND: track 116.4 -> 91.4 mm
- net +5V: track 55.9 -> 63.5 mm
- net Net-(D11-Pad1): track 16.3 -> 22.9 mm, vias 2 -> 0
- net Net-(Q7-Pad3): track 0.00 -> 5.08 mm
- net Net-(Q5-Pad3): track 0.00 -> 5.02 mm
- net Carry: track 0.00 -> 2.54 mm
- net Net-(Q7-Pad2): track 0.00 -> 2.54 mm
- net Net-(Q5-Pad2): track 0.00 -> 2.54 mm
- net Net-(D13-Pad2): track 7.62 -> 10.2 mm
- net Net-(D10-Pad2): track 7.62 -> 10.2 mm
